File: Hardware/eagle_files/powerpack.brd (EAGLE design)
At the start: 68.2 x 45.7 mm, 15 parts, among them IC2 7805TV, Q1 IRLZ44Z

Commit message: blubb
Parts:
- moved POWER 1.91 mm to (21.6, 36.2), turned to 180 degrees
- moved PUMP 1.91 mm to (10.2, 36.2), turned to 180 degrees
- moved FLOW 1.27 mm to (7.62, 6.35)
- moved IC2 1.27 mm to (58.4, 3.81)
- renumbered TO_CTRL_BOX to VALVES, X3 to CTRL
Connections:
- net +12V: now also POWER.2, PUMP.1; no longer POWER.1, PUMP.2
- net GND: now also POWER.1; no longer POWER.2
- net N$15: now also PUMP.2; no longer PUMP.1
Routing:
- net N$1: track 14.8 -> 12.1 mm
- net N$15: track 41.0 -> 42.5 mm
- net N$12: track 14.9 -> 16.1 mm
- net N$2: track 7.99 -> 8.73 mm
