File: Hardware/eagle_files/powerpack.sch (EAGLE design)
At the start: 11 parts, among them IC2 7805TV, Q1 IRLZ44Z

Commit message: Powerpack Eagle File
Parts:
- removed X1: (no value), con-wago-500:W237-102
- removed X2: (no value), con-wago-500:W237-103
- added FLOW: (no value), con-wago-508:W237-03P
- added IC3: (no value), uln-udn:ULN2803A
- added JP1: (no value), pinhead:PINHD-1X2
- added POWER, PUMP: (no value), con-wago-500:W237-102
- added TO_CTRL_BOX: (no value), con-wago-508:W237-07P
Connections:
- removed net N$17: X1-2.KL
- removed net N$5: D2.A, IC1.GND, Q1.S
- new net +12V: D1.A, FLOW-1.KL, IC1.CD+, IC3.CD+, POWER-1.KL, PUMP-2.KL, TO_CTRL_BOX-7.KL
- new net +5V: C2.+, IC2.VO, X3.B-1
- new net GND: C1.-, C2.-, D2.A, IC1.GND, IC2.GND, IC3.GND, POWER-2.KL, Q1.S, X3.B-2
- new net N$16: IC3.O1, IC3.O2, TO_CTRL_BOX-4.KL
- new net N$18: IC3.O3, IC3.O4, TO_CTRL_BOX-3.KL
- new net N$19: IC3.O5, IC3.O6, TO_CTRL_BOX-2.KL
- new net N$20: IC3.O7, IC3.O8, TO_CTRL_BOX-1.KL
- new net N$21: IC3.I7, IC3.I8, X3.B-3
- new net N$22: IC3.I5, IC3.I6, X3.B-4
- new net N$23: IC3.I3, IC3.I4, X3.B-5
- new net N$24: IC3.I1, IC3.I2, X3.B-6
- new net N$26: R1.1, X3.B-9
- net N$12: now also TO_CTRL_BOX-6.KL
- net N$13: now also TO_CTRL_BOX-5.KL
- net N$15: now also FLOW-2.KL, PUMP-1.KL; no longer X1-1.KL
- net N$2: now also FLOW-3.KL, X3.B-12; no longer C1.-, C2.-, IC2.GND
- net N$3: now also JP1.1, X3.B-11; no longer D1.A
- net N$4: now also JP1.2, X3.B-10; no longer C2.+, IC2.VO
- net N$8: now also X3.B-8
- net N$9: now also X3.B-7
Other:
- moved on the sheet: C1, C2, D1, D2, IC1, IC2, Q1, R1, X3

Commit message: blubb
Parts:
- renumbered TO_CTRL_BOX to VALVES, X3 to CTRL
Connections:
- net +12V: now also POWER-2.KL, PUMP-1.KL; no longer POWER-1.KL, PUMP-2.KL
- net GND: now also POWER-1.KL; no longer POWER-2.KL
- net N$15: now also PUMP-2.KL; no longer PUMP-1.KL
Other:
- moved on the sheet: POWER-1, POWER-2, PUMP-1, PUMP-2
