File: hardware/eagle_files/powerpack.brd (EAGLE design)
At the start: 68.2 x 45.7 mm, 15 parts, among them IC2 7805TV, Q1 IRLZ44Z

Commit message: Version 1.0
Parts:
- moved Q1 2.54 mm to (10.2, 8.89)
Routing:
- net GND: track 136.8 -> 139.3 mm
- net N$14: track 3.96 -> 5.01 mm
- added copper zone on layer 16, net N$5
Other:
- board outline removed
- board text removed: "Tomatron PowerPack"
Changed lines of the file:
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@@
 <board>
 <plain>
-<wire x1="0" y1="0" x2="68.25" y2="0" width="0" layer="20"/>
-<wire x1="68.25" y1="0" x2="68.25" y2="45.71" width="0" layer="20"/>
-<wire x1="68.25" y1="45.71" x2="0" y2="45.71" width="0" layer="20"/>
-<wire x1="0" y1="45.71" x2="0" y2="0" width="0" layer="20"/>
-<text x="66.04" y="40.64" size="2.54" layer="16" rot="MR0">Tomatron PowerPack</text>
 </plain>
 <attributes>
@@
 <element name="IC3" library="uln-udn" package="DIL18" value="" x="52.07" y="25.4"/>
 <element name="JP1" library="pinhead" package="1X02" value="" x="22.86" y="15.24"/>
-<element name="Q1" library="transistor-power" package="TO220BH" value="IRLZ44Z" x="10.16" y="11.43" rot="R180"/>
+<element name="Q1" library="transistor-power" package="TO220BH" value="IRLZ44Z" x="10.16" y="8.89" rot="R180"/>
 <element name="R1" library="eagle-ltspice" package="0207/10" value="1,2k" x="21.59" y="18.415" rot="R180">
 <attribute name="SPICEPREFIX" value="R" x="21.59" y="18.415" size="1.778" layer="27" rot="R180" display="off"/>
@@
 <contactref element="Q1" pad="G"/>
 <wire x1="16.51" y1="18.415" x2="15.24" y2="17.78" width="1.4224" layer="16"/>
-<wire x1="15.24" y1="17.78" x2="12.7" y2="17.78" width="1.4224" layer="16"/>
+<wire x1="15.24" y1="17.78" x2="12.7" y2="15.24" width="1.4224" layer="16"/>
 </signal>
 <signal name="N$15">
@@
 <wire x1="7.62" y1="31.75" x2="6.35" y2="31.75" width="2.1844" layer="16"/>
 <wire x1="6.35" y1="31.75" x2="5.08" y2="30.48" width="2.1844" layer="16"/>
-<wire x1="5.08" y1="30.48" x2="5.08" y2="13.97" width="2.1844" layer="16"/>
-<wire x1="5.08" y1="13.97" x2="7.62" y2="13.97" width="2.1844" layer="16"/>
-<wire x1="7.62" y1="13.97" x2="10.16" y2="13.97" width="2.1844" layer="16"/>
-<wire x1="10.16" y1="13.97" x2="10.16" y2="17.78" width="2.1844" layer="16"/>
-<wire x1="7.62" y1="5.715" x2="7.62" y2="13.97" width="2.1844" layer="16"/>
+<wire x1="5.08" y1="30.48" x2="5.08" y2="11.43" width="2.1844" layer="16"/>
+<wire x1="5.08" y1="11.43" x2="7.62" y2="8.89" width="2.1844" layer="16"/>
+<wire x1="7.62" y1="8.89" x2="10.16" y2="11.43" width="2.1844" layer="16"/>
+<wire x1="10.16" y1="11.43" x2="10.16" y2="15.24" width="2.1844" layer="16"/>
+<wire x1="7.62" y1="5.715" x2="7.62" y2="8.89" width="2.1844" layer="16"/>
 </signal>
 <signal name="N$16">
@@
 <wire x1="24.09" y1="37.465" x2="24.13" y2="37.465" width="0.4064" layer="16"/>
 <wire x1="24.13" y1="37.465" x2="24.13" y2="36.83" width="0.4064" layer="16"/>
-<wire x1="7.62" y1="17.78" x2="7.62" y2="21.59" width="2.1844" layer="16"/>
+<wire x1="7.62" y1="15.24" x2="7.62" y2="21.59" width="2.1844" layer="16"/>
 <wire x1="7.62" y1="21.59" x2="10.16" y2="24.13" width="2.1844" layer="16"/>
 <wire x1="10.16" y1="24.13" x2="10.16" y2="41.275" width="2.1844" layer="16"/>
@@
 <wire x1="21.77" y1="8.85" x2="21.59" y2="15.24" width="0.8128" layer="16"/>
 </signal>
+<signal name="N$5">
+<polygon width="0.4064" layer="16" spacing="0.6096" isolate="0.6096">
+<vertex x="-6.35" y="49.53"/>
+<vertex x="73.66" y="49.53"/>
+<vertex x="73.66" y="-8.89"/>
+<vertex x="-6.35" y="-8.89"/>
+</polygon>
+</signal>
 </signals>
